File: power train/power train2.kicad_pcb (KiCad board)
At the start: 2 copper layers, 57.5 x 49.5 mm, 16 parts, among them J1 Conn_01x01_Pin, J3 Conn_01x01_Pin, J4 Conn_01x01_Pin, J5 Conn_01x01_Pin, J6 Conn_01x01_Pin, J7 Conn_01x01_Pin, Q1 160N60UFD, U1 NSL-32

Commit message: power train
Parts:
- moved J6 40.0 mm to (108.8, 58.4)
- moved R3 15.1 mm to (88.2, 73.0)
- moved C4 5.14 mm to (100.6, 76.8), turned to -90 degrees
- moved J3 4.60 mm to (129.8, 58.4)
- moved J4 4.60 mm to (129.8, 61.4)
- moved VLA1 4.52 mm to (124.0, 76.2)
- moved J5 2.60 mm to (112.6, 58.4)
- moved C1 1.95 mm to (112.5, 91.0), turned to 180 degrees
Routing:
- net Net-(U1-K): track 48.5 -> 97.1 mm, vias 1 -> 0
- net +20V: track 81.9 -> 56.4 mm
- net Net-(U1-A): track 31.0 -> 7.73 mm
- net GND: track 57.2 -> 35.4 mm
- net Net-(J6-Pin_1): track 71.8 -> 58.7 mm
- net Net-(D1-A): track 27.3 -> 30.7 mm
- net Net-(VLA1-Gate): track 75.4 -> 78.3 mm
