File: power train/power train2.kicad_sch (KiCad schematic)
At the start: 16 parts, among them J1 Conn_01x01_Pin, J3 Conn_01x01_Pin, J4 Conn_01x01_Pin, J5 Conn_01x01_Pin, J6 Conn_01x01_Pin, J7 Conn_01x01_Pin, Q1 160N60UFD, U1 NSL-32

Commit message: power train
Changed lines of the file:
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@@
 				)
 				(justify left)
+				(hide yes)
 			)
 		)
@@
 			)
 		)
-		(property "Description" ""
+		(property "Description" "160A, 600V, N-Channel IGBT"
 			(at 142.24 93.98 0)
 			(effects
